File: macrosKeyboard/macrosKeyboard.kicad_sch (KiCad schematic)
At the start: 32 parts, among them J1 USB_B_Micro, J2 Conn_01x03_Male, SW1 PTS815_SJM_250_SMTR_LFS, U1 RP2040, U2 AMS1117, U3 W25Q128JVS, Y1 Crystal

Commit message: test change of naem
Other:
- company: everyday dev -> Huskies' lab
- title: PROJECT_TITLE_HERE -> siberianMacrosKeyboard
